Commit message: controller

File: src/robot_body/urdf/gazebo_control.xacro (robot description, xacro)
@@ -2,6 +2,10 @@
 <robot xmlns:xacro="http://www.ros.org/wiki/xacro" >
     <gazebo>
-        <plugin name="diff_drive" filename="libgazebo_ros_diffdrive.so">
+        <plugin name="diff_drive" filename="libgazebo_ros_diff_drive.so">
             <!-- <robotNamespace>/autoJetsonBot</robotNamespace> -->
+            <ros>
+                <namespace>/</namespace>
+                <remapping>cmd_vel:=/cmd_vel</remapping>
+            </ros>
             <!-- wheel info -->
             <left_joint>left_wheel_joint</left_joint>
@@ -9,8 +13,9 @@
             <caster_wheel_joint>caster_wheel_joint</caster_wheel_joint>
             <wheel_separation>0.15</wheel_separation>
+            <wheel_diameter>0.07</wheel_diameter>
             <wheel_radius>0.035</wheel_radius>
             <!-- limits -->
-            <max_wheel_torque>50.0</max_wheel_torque>
-            <max_wheel_acceleration>5</max_wheel_acceleration>
+            <max_wheel_torque>250.0</max_wheel_torque>
+            <max_wheel_acceleration>25</max_wheel_acceleration>
             <!-- output -->
             <odametry_frame>odom</odametry_frame>

File: src/robot_body/urdf/robot.xacro (robot description, xacro)
@@ -10,3 +10,6 @@
     <xacro:include filename="robot_core.xacro" />
     <xacro:include filename="gazebo_control.xacro" />
+    <xacro:include filename="lidar.xacro" />
+    <xacro:include filename="camera.xacro" />
+    <xacro:include filename="ros2_control.xacro" />
 </robot>

File: src/robot_body/urdf/robot_core.xacro (robot description, xacro)
@@ -1,5 +1,5 @@
 <?xml version="1.0"?>
 <robot xmlns:xacro="http://www.ros.org/wiki/xacro" >
-<xacro:property name="pi" value="3.14159265359"/>
+<!-- <xacro:property name="pi" value="3.14159265359"/>    -->
 <xacro:include filename="inertial_macros.xacro" />
     <!-- COLORS FOR ROBOT PARTS -->
@@ -150,6 +150,6 @@
     <!-- ROBOT LIDAR -->
     <joint name="lidar_joint" type="fixed">
-        <origin xyz="0.035 0 0.07" rpy="0 0 0"/>
-        <parent link="base_link"/>
+        <origin xyz="0.07 0 0.07" rpy="0 0 0"/>
+        <parent link="chassis"/>
         <child link="lidar"/>
     </joint>
