Commit message: slam

File: src/my_robot_launch/urdf/lidar.xacro (robot description, xacro)
@@ -56,5 +56,6 @@
                     <!-- <argument>~/out:=/scan</argument> -->
                     <!-- <argument> remapping:=/scan:=/scan</argument>    -->
-                    <argument>scan:=/scan</argument>
+                    <!-- <argument>scan:=/scan</argument> -->
+                    <argument>--ros-args --remap scan:=/scan</argument>
                 </ros>
                 <!-- <topicName>scan</topicName> -->

File: src/my_robot_launch/urdf/robot_core.xacro (robot description, xacro)
@@ -35,5 +35,5 @@
     <link name="base_link">
     </link>
-    </link>
+    <!-- </link> -->
     <!-- BASE_FOOTPRINT LINK -->
     <joint name="base_footprint_joint" type="fixed">

File: src/my_robot_launch/urdf/ros2_control.xacro (robot description, xacro)
@@ -1,4 +1,4 @@
 <?xml version="1.0"?>
-<!-- autoJetsonBot/src/robot_body/urdf/ros2_control.xacro -->
+<!-- autoJetsonBot/src/my_robot_launch/urdf/ros2_control.xacro -->
 <robot xmlns:xacro="http://www.ros.org/wiki/xacro">
     <xacro:unless value="$(arg sim_mode)">
@@ -56,6 +56,6 @@
         <gazebo>
             <plugin name="gazebo_ros2_control" filename="libgazebo_ros2_control.so">
-                <parameters>$(find robot_body)/config/my_controllers.yaml</parameters>
-                <parameters>$(find robot_body)/config/gaz_ros2_ctl_use_sim.yaml</parameters>
+                <parameters>$(find my_robot_launch)/config/my_controllers.yaml</parameters>
+                <parameters>$(find my_robot_launch)/config/gaz_ros2_ctl_use_sim.yaml</parameters>
             </plugin>
         </gazebo>

Commit message: slam

File: src/my_robot_launch/urdf/lidar.xacro (robot description, xacro)
@@ -1,34 +1,38 @@
 <?xml version="1.0"?>
 <robot xmlns:xacro="http://www.ros.org/wiki/xacro" >
-    <!-- laser -->
+<!-- /home/jetson/myspace/autoJetsonBot/src/my_robot_launch/urdf/lidar.xacro -->
     <joint name="laser_joint" type="fixed">
-        <!-- <origin xyz="-0.03 0 0" rpy="0 0 0"/> -->
-        <origin xyz="0.07 0 0.07" rpy="0 0 0"/>
         <parent link="chassis"/>
         <child link="laser_frame"/>
+        <origin xyz="0.1 0 0.135" rpy="0 0 0"/>
     </joint>
     <link name="laser_frame">
         <visual>
-            <origin xyz="0 0 0" rpy="0 0 0"/>
             <geometry>
-                <!-- <cylinder radius="0.02" length="0.01"/> -->
-                <cylinder radius="0.035" length="0.065"/>
+                <cylinder radius="0.05" length="0.04"/>
             </geometry>
-            <material name="red"/>
+            <material name="black"/>
+        </visual>
+        <visual>
+            <origin xyz="0 0 -0.05"/>
+            <geometry>
+                <cylinder radius="0.01" length="0.1"/>
+            </geometry>
+            <material name="black"/>
         </visual>
         <collision>
-            <origin xyz="0 0 0" rpy="0 0 0"/>
             <geometry>
-                <cylinder radius="0.035" length="0.065"/>
+                <cylinder radius="0.05" length="0.04"/>
             </geometry>
         </collision>
-        <xacro:inertial_cylinder mass="0.1" radius="0.035" length="0.065">
+        <xacro:inertial_cylinder mass="0.1" length="0.04" radius="0.05">
             <origin xyz="0 0 0" rpy="0 0 0"/>
         </xacro:inertial_cylinder>
     </link>
     <gazebo reference="laser_frame">
+        <material>Gazebo/Black</material>
         <sensor name="laser" type="ray">
-            <pose>0 0 0 0 0 0</pose>
-            <visualize>true</visualize>
+            <pose> 0 0 0 0 0 0 </pose>
+            <visualize>false</visualize>
             <update_rate>10</update_rate>
             <ray>
@@ -36,5 +40,4 @@
                     <horizontal>
                         <samples>360</samples>
-                        <resolution>1</resolution>
                         <min_angle>-3.14</min_angle>
                         <max_angle>3.14</max_angle>
@@ -42,27 +45,16 @@
                 </scan>
                 <range>
-                    <min>0.2</min>
+                    <min>0.3</min>
                     <max>12</max>
-                    <resolution>0.01</resolution>
                 </range>
-                <noise>
-                    <type>gaussian</type>
-                    <mean>0.0</mean>
-                    <stddev>0.01</stddev>
-                </noise>
             </ray>
-            <plugin name="gazebo_ros_laser" filename="libgazebo_ros_ray_sensor.so">
+            <plugin name="laser_controller" filename="libgazebo_ros_ray_sensor.so">
                 <ros>
-                    <!-- <argument>~/out:=/scan</argument> -->
-                    <!-- <argument> remapping:=/scan:=/scan</argument>    -->
-                    <!-- <argument>scan:=/scan</argument> -->
-                    <argument>--ros-args --remap scan:=/scan</argument>
+                    <argument>~/out:=scan</argument>
                 </ros>
-                <!-- <topicName>scan</topicName> -->
-                <frameName>laser_frame</frameName>
                 <output_type>sensor_msgs/LaserScan</output_type>
+                <frame_name>laser_frame</frame_name>
             </plugin>
         </sensor>
-        <material>Gazebo/Red</material>
     </gazebo>
 </robot>

File: src/my_robot_launch/urdf/robot.xacro (robot description, xacro)
@@ -5,13 +5,13 @@
     <xacro:arg name="sim_mode" default="false"/>
     <xacro:include filename="robot_core.xacro" />
-    <xacro:include filename="ros2_control.xacro" />
-    <!-- <xacro:if value="$(arg use_ros2_control)">
+    <xacro:if value="$(arg use_ros2_control)">
         <xacro:include filename="ros2_control.xacro" />
     </xacro:if>
     <xacro:unless value="$(arg use_ros2_control)">
         <xacro:include filename="gazebo_control.xacro" />
-    </xacro:unless> -->
+    </xacro:unless>
     <xacro:include filename="lidar.xacro" />
     <xacro:include filename="camera.xacro" />
     <!-- <xacro:include filename="depth_camera.xacro" /> -->
+    <!-- <xacro:include filename="face.xacro" /> -->
 </robot>

File: src/my_robot_launch/urdf/robot_core copy.xacro (robot description, xacro)
@@ -75,5 +75,5 @@
     <!-- LEFT WHEEL -->
     <joint name="left_wheel_joint" type="continuous">
-        <origin xyz="0 0.09 -0.02" rpy="-${pi/2} 0 0"/>
+        <origin xyz="0 0.105 -0.02" rpy="-${pi/2} 0 0"/>
         <parent link="base_link"/>
         <child link="left_wheel"/>
@@ -103,5 +103,5 @@
     <!-- RIGHT WHEEL -->
     <joint name="right_wheel_joint" type="continuous">
-        <origin xyz="0 -0.09 -0.02" rpy="${pi/2} 0 0"/>
+        <origin xyz="0 -0.105 -0.02" rpy="${pi/2} 0 0"/>
         <parent link="base_link"/>
         <child link="right_wheel"/>

File: src/my_robot_launch/urdf/robot_core.xacro (robot description, xacro)
@@ -7,4 +7,7 @@
     <material name="grey">
         <color rgba="0.5 0.5 0.5 1"/>
+    </material>
+        <material name="grey2">
+        <color rgba="0.75 0.75 0.75 1"/>
     </material>
     <material name="red">
@@ -46,5 +49,5 @@
     <!-- ROBOT CHASSIS LINK-->
     <joint name="chassis_joint" type="fixed">
-        <origin xyz="-0.03 0 0" rpy="0 0 0"/>
+        <origin xyz="-0.035 0 0" rpy="0 0 0"/>
         <parent link="base_link"/>
         <child link="chassis"/>
@@ -53,18 +56,18 @@
     <link name="chassis">
         <visual>
-            <origin xyz="0.0725 0 0.035" rpy="0 0 0"/>
+            <origin xyz="0.0975 0 0.05" rpy="0 0 0"/>
             <geometry>
-                <box size="0.145 0.14 0.07"/>
+                <box size="0.195 0.18 0.1"/>
             </geometry>
-            <material name="white"/>
+            <material name="purple"/>
         </visual>
         <collision>
-            <origin xyz="0.0725 0 0.035" rpy="0 0 0"/>
+            <origin xyz="0.0975 0 0.05" rpy="0 0 0"/>
             <geometry>
-                <box size="0.145 0.14 0.07"/>
+                <box size="0.195 0.18 0.1"/>
             </geometry>
         </collision>
-        <xacro:inertial_box mass="0.5" x="0.145" y="0.14" z="0.07">
-            <origin xyz="0.0725 0 0.035" rpy="0 0 0"/>
+        <xacro:inertial_box mass="0.8" x="0.195" y="0.18" z="0.1">
+            <origin xyz="0.0975 0 0.05" rpy="0 0 0"/>
         </xacro:inertial_box>
     </link>
@@ -131,5 +134,5 @@
     <!-- CASTER WHEEL -->
     <joint name="caster_wheel_joint" type="fixed">
-        <origin xyz="0.095 0 -0.02" rpy="0 0 0"/>
+        <origin xyz="0.12 0 -0.02" rpy="0 0 0"/>
         <parent link="base_link"/>
         <child link="caster_wheel"/>
@@ -141,5 +144,5 @@
                 <sphere radius="0.035"/>
             </geometry>
-            <material name="black"/>
+            <material name="grey"/>
         </visual>
         <collision>
@@ -158,7 +161,7 @@
         <mu2 value="0.001"/>
     </gazebo>
-    <!-- ROBOT LIDAR -->
+    <!-- ROBOT LIDAR
     <joint name="lidar_joint" type="fixed">
-        <origin xyz="0.07 0 0.07" rpy="0 0 0"/>
+        <origin xyz="0.1 0 0.135" rpy="0 0 0"/>
         <parent link="chassis"/>
         <child link="lidar"/>
@@ -181,5 +184,5 @@
     <gazebo reference="lidar">
         <material>Gazebo/Red</material>
-    </gazebo>
+    </gazebo> -->
 </robot>
 <!--

File: src/my_robot_launch/urdf/ros2_control.xacro (robot description, xacro)
@@ -8,5 +8,5 @@
                 <param name="left_wheel_name">left_wheel_joint</param>
                 <param name="right_wheel_name">right_wheel_joint</param>
-                <param name="loop_rate">30</param>
+                <param name="loop_rate">60</param>
                 <param name="device">/dev/ttyACM0</param>  <!-- or whichever device you found -->
                 <param name="baud_rate">115200</param>
@@ -17,5 +17,5 @@
                 <command_interface name="velocity">
                     <param name="min">-10</param>
-                    <param name="max">10</param>
+                    <param name="max">50</param>
                 </command_interface>
                 <state_interface name="velocity"/>
@@ -25,5 +25,5 @@
                 <command_interface name="velocity">
                     <param name="min">-10</param>
-                    <param name="max">10</param>
+                    <param name="max">50</param>
                 </command_interface>
                 <state_interface name="velocity"/>
@@ -40,5 +40,5 @@
                 <command_interface name="velocity">
                     <param name="min">-10</param>
-                    <param name="max">10</param>
+                    <param name="max">50</param>
                 </command_interface>
                 <state_interface name="velocity"/>
@@ -48,5 +48,5 @@
                 <command_interface name="velocity">
                     <param name="min">-10</param>
-                    <param name="max">10</param>
+                    <param name="max">50</param>
                 </command_interface>
                 <state_interface name="velocity"/>
