Commit message: slam

File: src/my_robot_launch/urdf/robot_core copy 2.xacro (robot description, xacro)
@@ -35,5 +35,5 @@
     <link name="base_link">
     </link>
-    </link>
+    <!-- </link> -->
     <!-- BASE_FOOTPRINT LINK -->
     <joint name="base_footprint_joint" type="fixed">
@@ -46,5 +46,5 @@
     <!-- ROBOT CHASSIS LINK-->
     <joint name="chassis_joint" type="fixed">
-        <origin xyz="-0.03 0 0" rpy="0 0 0"/>
+        <origin xyz="-0.035 0 0" rpy="0 0 0"/>
         <parent link="base_link"/>
         <child link="chassis"/>
@@ -53,18 +53,18 @@
     <link name="chassis">
         <visual>
-            <origin xyz="0.0725 0 0.035" rpy="0 0 0"/>
+            <origin xyz="0.0975 0 0.05" rpy="0 0 0"/>
             <geometry>
-                <box size="0.145 0.14 0.07"/>
+                <box size="0.195 0.18 0.1"/>
             </geometry>
-            <material name="white"/>
+            <material name="gray"/>
         </visual>
         <collision>
-            <origin xyz="0.0725 0 0.035" rpy="0 0 0"/>
+            <origin xyz="0.0975 0 0.05" rpy="0 0 0"/>
             <geometry>
-                <box size="0.145 0.14 0.07"/>
+                <box size="0.195 0.18 0.1"/>
             </geometry>
         </collision>
-        <xacro:inertial_box mass="0.5" x="0.145" y="0.14" z="0.07">
-            <origin xyz="0.0725 0 0.035" rpy="0 0 0"/>
+        <xacro:inertial_box mass="0.8" x="0.195" y="0.18" z="0.1">
+            <origin xyz="0.0975 0 0.05" rpy="0 0 0"/>
         </xacro:inertial_box>
     </link>
@@ -75,5 +75,5 @@
     <!-- LEFT WHEEL -->
     <joint name="left_wheel_joint" type="continuous">
-        <origin xyz="0 0.105 -0.02" rpy="-${pi/2} 0 0"/>
+        <origin xyz="0 0.09 -0.02" rpy="-${pi/2} 0 0"/>
         <parent link="base_link"/>
         <child link="left_wheel"/>
@@ -103,5 +103,5 @@
     <!-- RIGHT WHEEL -->
     <joint name="right_wheel_joint" type="continuous">
-        <origin xyz="0 -0.105 -0.02" rpy="${pi/2} 0 0"/>
+        <origin xyz="0 -0.09 -0.02" rpy="${pi/2} 0 0"/>
         <parent link="base_link"/>
         <child link="right_wheel"/>
