Commit message: nav2

File: src/jetson_bot_description/urdf/robot.xacro (robot description, xacro)
@@ -13,4 +13,5 @@
     <xacro:include filename="lidar.xacro" />
     <xacro:include filename="camera.xacro" />
+    <xacro:include filename="imu.xacro" />
     <!-- <xacro:include filename="depth_camera.xacro" /> -->
     <!-- <xacro:include filename="face.xacro" /> -->

File: src/jetson_bot_description/urdf/robot_core.xacro (robot description, xacro)
@@ -35,15 +35,14 @@
         <color rgba="1 1 1 1"/>
     </material>
-    <!-- ROBOT BASE LINK -->
+    <!-- BASE_FOOTPRINT LINK (The Floor Projection) -->
+    <link name="base_footprint">
+    </link>
+    <joint name="base_footprint_joint" type="fixed">
+        <parent link="base_footprint"/>
+        <child link="base_link"/>
+        <origin xyz="0 0 0.055" rpy="0 0 0"/>
+    </joint>
+    <!-- ROBOT BASE LINK (The Center of the Wheels) -->
     <link name="base_link">
-    </link>
-    <!-- </link> -->
-    <!-- BASE_FOOTPRINT LINK -->
-    <joint name="base_footprint_joint" type="fixed">
-        <parent link="base_link"/>
-        <child link="base_footprint"/>
-        <origin xyz="0 0 0" rpy="0 0 0"/>
-    </joint>
-    <link name="base_footprint">
     </link>
     <!-- ROBOT CHASSIS LINK-->
@@ -103,4 +102,8 @@
     <gazebo reference="left_wheel">
         <material>Gazebo/Black</material>
+        <mu1 value="100.0"/>
+        <mu2 value="100.0"/>
+        <kp value="1000000.0" />
+        <kd value="1.0" />
     </gazebo>
     <!-- RIGHT WHEEL -->
@@ -131,4 +134,8 @@
     <gazebo reference="right_wheel">
         <material>Gazebo/Black</material>
+        <mu1 value="100.0"/>
+        <mu2 value="100.0"/>
+        <kp value="1000000.0" />
+        <kd value="1.0" />
     </gazebo>
     <!-- CASTER WHEEL -->

File: src/jetson_bot_description/urdf/ros2_control.xacro (robot description, xacro)
@@ -57,4 +57,8 @@
             <plugin name="gazebo_ros2_control" filename="libgazebo_ros2_control.so">
                 <parameters>$(find jetson_bot_bringup)/config/unified_robot_config.yaml</parameters>
+                <ros>
+                    <remapping>/diff_cont/cmd_vel_unstamped:=/cmd_vel</remapping>
+                    <remapping>/diff_cont/odom:=/odom</remapping>
+                </ros>
             </plugin>
         </gazebo>
