Commit message: nav2 ui upgrade / physics simulation opt

File: src/jetson_bot_description/urdf/camera.xacro (robot description, xacro)
@@ -16,10 +16,4 @@
             <material name="red"/>
         </visual>
-        <collision>
-            <origin xyz="0 0 0" rpy="0 0 0"/>
-            <geometry>
-                <cylinder radius="0.035" length="0.025"/>
-            </geometry>
-        </collision>
         <xacro:inertial_cylinder mass="0.1" radius="0.035" length="0.025">
             <origin xyz="0 0 0" rpy="0 0 0"/>

File: src/jetson_bot_description/urdf/robot_core.xacro (robot description, xacro)
@@ -77,5 +77,5 @@
     <!-- LEFT WHEEL -->
     <joint name="left_wheel_joint" type="continuous">
-        <origin xyz="0 0.09 -0.02" rpy="-${pi/2} 0 0"/>
+        <origin xyz="0 0.11 -0.02" rpy="-${pi/2} 0 0"/>
         <parent link="base_link"/>
         <child link="left_wheel"/>
@@ -86,5 +86,5 @@
             <origin xyz="0 0 0" rpy="0 0 0"/>
             <geometry>
-                <cylinder radius="0.035" length="0.027"/>
+                <cylinder radius="0.035" length="0.026"/>
             </geometry>
             <material name="black"/>
@@ -93,8 +93,8 @@
             <origin xyz="0 0 0" rpy="0 0 0"/>
             <geometry>
-                <cylinder radius="0.035" length="0.027"/>
+                <cylinder radius="0.035" length="0.026"/>
             </geometry>
         </collision>
-        <xacro:inertial_cylinder mass="0.1" length="0.027" radius="0.035">
+        <xacro:inertial_cylinder mass="0.1" length="0.026" radius="0.035">
             <origin xyz="0 0 0" rpy="0 0 0"/>
         </xacro:inertial_cylinder>
@@ -109,5 +109,5 @@
     <!-- RIGHT WHEEL -->
     <joint name="right_wheel_joint" type="continuous">
-        <origin xyz="0 -0.09 -0.02" rpy="${pi/2} 0 0"/>
+        <origin xyz="0 -0.11 -0.02" rpy="${pi/2} 0 0"/>
         <parent link="base_link"/>
         <child link="right_wheel"/>
@@ -118,5 +118,5 @@
             <origin xyz="0 0 0" rpy="0 0 0"/>
             <geometry>
-                <cylinder radius="0.035" length="0.025"/>
+                <cylinder radius="0.035" length="0.026"/>
             </geometry>
             <material name="black"/>
@@ -125,8 +125,8 @@
             <origin xyz="0 0 0" rpy="0 0 0"/>
             <geometry>
-                <cylinder radius="0.035" length="0.025"/>
+                <cylinder radius="0.035" length="0.026"/>
             </geometry>
         </collision>
-        <xacro:inertial_cylinder mass="0.1" length="0.025" radius="0.035">
+        <xacro:inertial_cylinder mass="0.1" length="0.026" radius="0.035">
             <origin xyz="0 0 0" rpy="0 0 0"/>
         </xacro:inertial_cylinder>
@@ -193,13 +193,2 @@
     </gazebo> -->
 </robot>
-<!--
-my robot dimensions:
-    base:
-        - center point between the wheels: 0 0 0 mm
-    chassis:
-        - length: 145 mm
-        - width: 140 mm
-        - height: 70  mm
-        - chassis_joint origin point: -30 0 0 mm (behind the center point between the wheels)
-        - chassis origin point: 72.5 0 35 mm (behind the center point between the wheels)
- -->
