Commit message: motor hardare deployment complete

File: src/jetson_bot_description/urdf/lidar.xacro (robot description, xacro)
@@ -5,5 +5,5 @@
         <parent link="chassis"/>
         <child link="laser_frame"/>
-        <origin xyz="0.1 0 0.135" rpy="0 0 0"/>
+        <origin xyz="0.064 0 0.161" rpy="0 0 0"/>
     </joint>
     <link name="laser_frame">

File: src/jetson_bot_description/urdf/robot_core.xacro (robot description, xacro)
@@ -41,12 +41,12 @@
         <parent link="base_footprint"/>
         <child link="base_link"/>
-        <origin xyz="0 0 0.055" rpy="0 0 0"/>
+        <origin xyz="0 0 0.056" rpy="0 0 0"/>
     </joint>
-    <!-- ROBOT BASE LINK (The Center of the Wheels) -->
+    <!-- ROBOT BASE LINK (The Center of the Chassis Floor) -->
     <link name="base_link">
     </link>
     <!-- ROBOT CHASSIS LINK-->
     <joint name="chassis_joint" type="fixed">
-        <origin xyz="-0.035 0 0" rpy="0 0 0"/>
+        <origin xyz="0 0 0" rpy="0 0 0"/>
         <parent link="base_link"/>
         <child link="chassis"/>
@@ -55,18 +55,18 @@
     <link name="chassis">
         <visual>
-            <origin xyz="0.0975 0 0.05" rpy="0 0 0"/>
+            <origin xyz="0.061 0 0.0485" rpy="0 0 0"/>
             <geometry>
-                <box size="0.195 0.18 0.1"/>
+                <box size="0.194 0.178 0.097"/>
             </geometry>
             <material name="purple"/>
         </visual>
         <collision>
-            <origin xyz="0.0975 0 0.05" rpy="0 0 0"/>
+            <origin xyz="0.061 0 0.0485" rpy="0 0 0"/>
             <geometry>
-                <box size="0.195 0.18 0.1"/>
+                <box size="0.194 0.178 0.097"/>
             </geometry>
         </collision>
-        <xacro:inertial_box mass="0.8" x="0.195" y="0.18" z="0.1">
-            <origin xyz="0.0975 0 0.05" rpy="0 0 0"/>
+        <xacro:inertial_box mass="1.2" x="0.194" y="0.178" z="0.097">
+            <origin xyz="0.061 0 0.0485" rpy="0 0 0"/>
         </xacro:inertial_box>
     </link>
@@ -77,5 +77,5 @@
     <!-- LEFT WHEEL -->
     <joint name="left_wheel_joint" type="continuous">
-        <origin xyz="0 0.11 -0.02" rpy="-${pi/2} 0 0"/>
+        <origin xyz="0 0.106 -0.022" rpy="-${pi/2} 0 0"/>
         <parent link="base_link"/>
         <child link="left_wheel"/>
@@ -86,5 +86,5 @@
             <origin xyz="0 0 0" rpy="0 0 0"/>
             <geometry>
-                <cylinder radius="0.035" length="0.026"/>
+                <cylinder radius="0.034" length="0.026"/>
             </geometry>
             <material name="black"/>
@@ -93,8 +93,8 @@
             <origin xyz="0 0 0" rpy="0 0 0"/>
             <geometry>
-                <cylinder radius="0.035" length="0.026"/>
+                <cylinder radius="0.034" length="0.026"/>
             </geometry>
         </collision>
-        <xacro:inertial_cylinder mass="0.1" length="0.026" radius="0.035">
+        <xacro:inertial_cylinder mass="0.1" length="0.026" radius="0.034">
             <origin xyz="0 0 0" rpy="0 0 0"/>
         </xacro:inertial_cylinder>
@@ -109,5 +109,5 @@
     <!-- RIGHT WHEEL -->
     <joint name="right_wheel_joint" type="continuous">
-        <origin xyz="0 -0.11 -0.02" rpy="${pi/2} 0 0"/>
+        <origin xyz="0 -0.106 -0.022" rpy="${pi/2} 0 0"/>
         <parent link="base_link"/>
         <child link="right_wheel"/>
@@ -118,5 +118,5 @@
             <origin xyz="0 0 0" rpy="0 0 0"/>
             <geometry>
-                <cylinder radius="0.035" length="0.026"/>
+                <cylinder radius="0.034" length="0.026"/>
             </geometry>
             <material name="black"/>
@@ -125,8 +125,8 @@
             <origin xyz="0 0 0" rpy="0 0 0"/>
             <geometry>
-                <cylinder radius="0.035" length="0.026"/>
+                <cylinder radius="0.034" length="0.026"/>
             </geometry>
         </collision>
-        <xacro:inertial_cylinder mass="0.1" length="0.026" radius="0.035">
+        <xacro:inertial_cylinder mass="0.1" length="0.026" radius="0.034">
             <origin xyz="0 0 0" rpy="0 0 0"/>
         </xacro:inertial_cylinder>
@@ -141,5 +141,5 @@
     <!-- CASTER WHEEL -->
     <joint name="caster_wheel_joint" type="fixed">
-        <origin xyz="0.12 0 -0.02" rpy="0 0 0"/>
+        <origin xyz="0.115 0 -0.022" rpy="0 0 0"/>
         <parent link="base_link"/>
         <child link="caster_wheel"/>
@@ -149,5 +149,5 @@
             <origin xyz="0 0 0" rpy="0 0 0"/>
             <geometry>
-                <sphere radius="0.035"/>
+                <sphere radius="0.034"/>
             </geometry>
             <material name="grey"/>
@@ -156,8 +156,8 @@
             <origin xyz="0 0 0" rpy="0 0 0"/>
             <geometry>
-                <sphere radius="0.035"/>
+                <sphere radius="0.034"/>
             </geometry>
         </collision>
-        <xacro:inertial_sphere mass="0.1" radius="0.035">
+        <xacro:inertial_sphere mass="0.1" radius="0.034">
             <origin xyz="0 0 0" rpy="0 0 0"/>
         </xacro:inertial_sphere>
