Commit message: simtry&realopt

File: src/jetson_bot_description/urdf/ros2_control.xacro (robot description, xacro)
@@ -3,32 +3,7 @@
 <robot xmlns:xacro="http://www.ros.org/wiki/xacro">
     <xacro:unless value="$(arg sim_mode)">
-        <ros2_control name="RealRobot" type="system">
-            <hardware>
-                <plugin>diffdrive_arduino/DiffDriveArduino</plugin>
-                <param name="left_wheel_name">left_wheel_joint</param>
-                <param name="right_wheel_name">right_wheel_joint</param>
-                <param name="loop_rate">60</param>
-                <param name="device">/dev/ttyACM0</param>  <!-- or whichever device you found -->
-                <param name="baud_rate">115200</param>
-                <param name="timeout">1000</param>
-                <param name="enc_counts_per_rev">3436</param>  <!-- STANDARDIZED - Phase 1 Migration -->
-            </hardware>
-            <joint name="left_wheel_joint">
-                <command_interface name="velocity">
-                    <param name="min">-10</param>
-                    <param name="max">50</param>
-                </command_interface>
-                <state_interface name="velocity"/>
-                <state_interface name="position"/>
-            </joint>
-            <joint name="right_wheel_joint">
-                <command_interface name="velocity">
-                    <param name="min">-10</param>
-                    <param name="max">50</param>
-                </command_interface>
-                <state_interface name="velocity"/>
-                <state_interface name="position"/>
-            </joint>
-        </ros2_control>
+        <!-- Hardware path uses standalone Python bridge (jetson_bot_diffdrive)
+             NOT the ros2_control hardware plugin. The old diffdrive_arduino plugin
+             is intentionally omitted here to prevent "plugin not found" issues. -->
     </xacro:unless>
     <xacro:if value="$(arg sim_mode)">
